Commit message: Rename throttled image topic

File: urdf/mltdma_mesh.xacro (robot description, xacro)
@@ -8,5 +8,5 @@
       <parent link="${namespace}/base_link"/>
       <child link="${namespace}/motion_sensor"/>
-      <origin xyz="0 0 0" rpy="0 0 0"/>
+      <origin xyz="0 0 0" rpy="0 0 1.5708"/>
   </joint>
   <link name="${namespace}/motion_sensor">
